File: anavi-opto-isolator.kicad_pcb (KiCad board)
At the start: 2 copper layers, 51.6 x 18.5 mm, 6 parts, among them J1 Screw_Terminal_01x02, J2 Screw_Terminal_01x03, U1 EL817

Commit message: anavi-opto-isolator: Add text on the back
Add text about open source hardware on the back of the printed
circuit board.

Signed-off-by: Leon Anavi <leon@anavi.org>
Other:
- board text added: "Open source hardware gives people the freedom to control their technology. https://anavi.technology/"
Changed lines of the file:
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@@
       (outputformat 1)
       (mirror false)
-      (drillshape 1)
+      (drillshape 0)
       (scaleselection 1)
-      (outputdirectory "")
+      (outputdirectory "plots/rev10/")
     )
   )
@@
     (fp_line (start -1 0.625) (end -1 -0.625) (layer "F.Fab") (width 0.1))
     (fp_line (start 1 0.625) (end -1 0.625) (layer "F.Fab") (width 0.1))
-    (pad "1" smd roundrect (at -1 0) (size 1.2 1.4) (layers "F.Cu" "F.Paste" "F.Mask") (roundrect_rratio 0.208333)
+    (pad "1" smd roundrect (at -1 0) (size 1.2 1.4) (layers "F.Cu" "F.Paste" "F.Mask") (roundrect_rratio 0.2083333333)
       (net 2 "+12V") (pintype "passive"))
-    (pad "2" smd roundrect (at 1 0) (size 1.2 1.4) (layers "F.Cu" "F.Paste" "F.Mask") (roundrect_rratio 0.208333)
+    (pad "2" smd roundrect (at 1 0) (size 1.2 1.4) (layers "F.Cu" "F.Paste" "F.Mask") (roundrect_rratio 0.2083333333)
       (net 6 "Net-(R1-Pad2)") (pintype "passive"))
     (model "${KICAD6_3DMODEL_DIR}/Resistor_SMD.3dshapes/R_0805_2012Metric.wrl"
@@
     (fp_line (start -1 0.625) (end -1 -0.625) (layer "F.Fab") (width 0.1))
     (fp_line (start -1 -0.625) (end 1 -0.625) (layer "F.Fab") (width 0.1))
-    (pad "1" smd roundrect (at -1 0 180) (size 1.2 1.4) (layers "F.Cu" "F.Paste" "F.Mask") (roundrect_rratio 0.208333)
+    (pad "1" smd roundrect (at -1 0 180) (size 1.2 1.4) (layers "F.Cu" "F.Paste" "F.Mask") (roundrect_rratio 0.2083333333)
       (net 3 "+3V3") (pintype "passive"))
-    (pad "2" smd roundrect (at 1 0 180) (size 1.2 1.4) (layers "F.Cu" "F.Paste" "F.Mask") (roundrect_rratio 0.208333)
+    (pad "2" smd roundrect (at 1 0 180) (size 1.2 1.4) (layers "F.Cu" "F.Paste" "F.Mask") (roundrect_rratio 0.2083333333)
       (net 4 "Net-(J2-Pad2)") (pintype "passive"))
     (model "${KICAD6_3DMODEL_DIR}/Resistor_SMD.3dshapes/R_0805_2012Metric.wrl"
@@
   (gr_line (start 65.786 48.26) (end 65.786 66.802) (layer "Edge.Cuts") (width 0.1))
   (gr_line (start 65.786 48.26) (end 117.348 48.26) (layer "Edge.Cuts") (width 0.1))
+  (gr_text "Open source hardware gives people the\nfreedom to control their technology.\n\nhttps://anavi.technology/" (at 91.44 57.15) (layer "B.SilkS")
+    (effects (font (size 1.2 1.2) (thickness 0.2)) (justify mirror))
+  )
   (gr_text "rev 1.0\n(c) 2024" (at 100.076 54.864) (layer "F.SilkS")
     (effects (font (size 0.6 0.6) (thickness 0.1)))
